File: eagle file/Square8_V1.3/Square8_V1.3.brd (EAGLE design)
At the start: 49.5 x 53 mm, 32 parts, among them J3 CR2032-172, Q1 si2305, U1 ATmega328mu, U2 CH340T, U3 CN3065, X1 16MHz, X2 12MHz

Commit message: update eagle file to 1.3, inprove the layout, expecially the RST line
Routing:
- net VCC: track 148.1 -> 167.8 mm
- net RESET: track 75.3 -> 62.5 mm, vias 2 -> 3
- net DTR: track 17.0 -> 20.9 mm
- net N$77: track 3.29 -> 0.00 mm
- net N$11: track 2.94 -> 0.00 mm
- net N$83: track 2.75 -> 0.00 mm
- net N$85: track 2.75 -> 0.00 mm
- net PD1/TX: track 5.75 -> 8.35 mm
- net COL1: track 36.4 -> 38.8 mm
- net ROW7: track 33.5 -> 35.8 mm
- net COL3: track 14.4 -> 16.6 mm
- net TX: track 21.8 -> 24.1 mm
- net RX: track 18.9 -> 21.2 mm
- net ROW4: track 13.9 -> 16.1 mm
- net ROW6: track 33.9 -> 36.1 mm
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Other:
- board text added: "V1.3 2014/5/15"
- board text removed: "V1.2 2014/4/30"
